File: PCB/Pico Bolt/pico servo.brd (EAGLE design)
At the start: 21.6 x 30.1 mm, 9 parts, among them J2 FEMALE 2x3, J3 FEMALE 2x3, J4 FEMALE 2x3, J5 FEMALE 2x3

Commit message: rz
no more car for now...
Parts:
- added ANALOG-IN: (no value), SparkFun-Connectors:1X06_NO_SILK
- moved C1 2.54 mm to (12.1, 29.2), turned to 180 degrees
Connections:
- net 3V: no longer C1.1
- net A0: now also ANALOG-IN.2
- net A1: now also ANALOG-IN.5
- net AG: now also ANALOG-IN.3, ANALOG-IN.4
- net AREF: now also ANALOG-IN.1, ANALOG-IN.6
- net V+: now also C1.1
Routing:
- net AREF: track 0.00 -> 17.3 mm
- net V+: track 30.5 -> 45.1 mm
- net A1: track 0.00 -> 6.55 mm
- net AG: track 0.00 -> 5.97 mm
- net 3V: track 3.83 -> 0.00 mm
- net A0: track 0.00 -> 3.43 mm
- net 5: track 9.31 -> 8.19 mm
Other:
- board text added: "G-"
- board text added: "PicoW x Bolt x10 Servo"
- board text added: "Saul C. 5/13/23 v1"
- board text added: "~3"
- board text added: "~4"
- board text added: "~5"
- board text added: "~6"
- board text removed: "CE28"
- board text removed: "RST"
