File: PCB/Pico Bolt/pico servo.sch (EAGLE design)
At the start: 9 parts, among them J2 FEMALE 2x3, J3 FEMALE 2x3, J4 FEMALE 2x3, J5 FEMALE 2x3

Commit message: rz
no more car for now...
Parts:
- added ANALOG-IN: (no value), SparkFun-Connectors:CONN_06NO_SILK_FEMALE_PTH
Connections:
- net 3V: no longer C1.+
- net A0: now also ANALOG-IN.2
- net A1: now also ANALOG-IN.5
- net AG: now also ANALOG-IN.3, ANALOG-IN.4
- net AREF: now also ANALOG-IN.1, ANALOG-IN.6
- net V+: now also C1.+
Changed lines of the file:
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@@
 <part name="J5" library="SparkFun-Connectors" deviceset="CONN_03X2" device="FEMALE" value="FEMALE 2x3"/>
 <part name="J4" library="SparkFun-Connectors" deviceset="CONN_03X2" device="FEMALE" value="FEMALE 2x3"/>
+<part name="ANALOG-IN" library="SparkFun-Connectors" deviceset="CONN_06" device="NO_SILK_FEMALE_PTH"/>
 </parts>
 <sheets>
@@
 <attribute name="VALUE" x="85.598" y="138.938" size="1.778" layer="96" font="vector" align="top-left"/>
 </instance>
+<instance part="ANALOG-IN" gate="JP1" x="124.46" y="76.2" smashed="yes">
+<attribute name="VALUE" x="119.38" y="66.294" size="1.778" layer="96" font="vector"/>
+<attribute name="NAME" x="119.38" y="86.868" size="1.778" layer="95" font="vector"/>
+</instance>
 </instances>
 <busses>
@@
 <pinref part="POWERSIDE" gate="G$1" pin="11"/>
 </segment>
+<segment>
+<pinref part="ANALOG-IN" gate="JP1" pin="6"/>
+<wire x1="129.54" y1="83.82" x2="137.16" y2="83.82" width="0.1524" layer="91"/>
+<label x="137.16" y="83.82" size="1.778" layer="95"/>
+</segment>
+<segment>
+<pinref part="ANALOG-IN" gate="JP1" pin="1"/>
+<wire x1="129.54" y1="71.12" x2="137.16" y2="71.12" width="0.1524" layer="91"/>
+<label x="137.16" y="71.12" size="1.778" layer="95"/>
+</segment>
 </net>
 <net name="3V" class="0">
@@
 <label x="50.8" y="30.48" size="1.778" layer="95"/>
 <pinref part="POWERSIDE" gate="G$1" pin="12"/>
-</segment>
-<segment>
-<pinref part="C1" gate="G$1" pin="+"/>
-<wire x1="88.9" y1="99.06" x2="81.28" y2="99.06" width="0.1524" layer="91"/>
-<wire x1="81.28" y1="99.06" x2="81.28" y2="88.9" width="0.1524" layer="91"/>
-<wire x1="81.28" y1="88.9" x2="76.2" y2="88.9" width="0.1524" layer="91"/>
-<label x="76.2" y="88.9" size="1.778" layer="95"/>
 </segment>
 </net>
@@
 <pinref part="POWERSIDE" gate="G$1" pin="9"/>
 </segment>
+<segment>
+<pinref part="ANALOG-IN" gate="JP1" pin="4"/>
+<wire x1="129.54" y1="78.74" x2="137.16" y2="78.74" width="0.1524" layer="91"/>
+<label x="137.16" y="78.74" size="1.778" layer="95"/>
+</segment>
+<segment>
+<pinref part="ANALOG-IN" gate="JP1" pin="3"/>
+<wire x1="129.54" y1="76.2" x2="137.16" y2="76.2" width="0.1524" layer="91"/>
+<label x="137.16" y="76.2" size="1.778" layer="95"/>
+</segment>
 </net>
 <net name="A1" class="0">
@@
 <pinref part="POWERSIDE" gate="G$1" pin="8"/>
 </segment>
+<segment>
+<pinref part="ANALOG-IN" gate="JP1" pin="5"/>
+<wire x1="129.54" y1="81.28" x2="137.16" y2="81.28" width="0.1524" layer="91"/>
+<label x="137.16" y="81.28" size="1.778" layer="95"/>
+</segment>
 </net>
 <net name="A0" class="0">
@@
 <label x="25.4" y="17.78" size="1.778" layer="95"/>
 <pinref part="POWERSIDE" gate="G$1" pin="7"/>
+</segment>
+<segment>
+<pinref part="ANALOG-IN" gate="JP1" pin="2"/>
+<wire x1="129.54" y1="73.66" x2="137.16" y2="73.66" width="0.1524" layer="91"/>
+<label x="137.16" y="73.66" size="1.778" layer="95"/>
 </segment>
 </net>
@@
 <pinref part="J4" gate="G$1" pin="4"/>
 </segment>
-</net>
+<segment>
+<pinref part="C1" gate="G$1" pin="+"/>
+<wire x1="88.9" y1="99.06" x2="81.28" y2="99.06" width="0.1524" layer="91"/>
+<wire x1="81.28" y1="99.06" x2="81.28" y2="88.9" width="0.1524" layer="91"/>
+<wire x1="81.28" y1="88.9" x2="76.2" y2="88.9" width="0.1524" layer="91"/>
+<label x="76.2" y="88.9" size="1.778" layer="95"/>
+</segment>
+</net>
